Commit message: blue_bot urdf

File: jazzy_ws/src/blue_bot/description/robot_core.xacro (robot description, xacro)
@@ -1,4 +1,5 @@
 <?xml version="1.0"?>
 <robot xmlns:xacro="http://www.ros.org/wiki/xacro">
+    <xacro:include filename="inertial_macros.xacro" />
     <!-- we'll define colors to use later-->
     <material name="white">
@@ -23,5 +24,5 @@
         <parent link="base_link"/>
         <child link="chassis"/>
-        <origin xyz="-0.1 0 0">
+        <origin xyz="0 0 0"/>
     </joint>
     <!-- Now we'll create the actual chassis link -->
@@ -35,4 +36,104 @@
             <material name="blue"/>
         </visual>
-    </chassis>
+        <collision>
+        <!-- The geometry will center in joint origin. We want to align it to the wheel connector -->
+            <origin xyz="0 0 0.0625"/>
+            <geometry>
+                <cylinder radius="0.08" length="0.125"/>
+            </geometry>
+        </collision>
+        <xacro:inertial_cylinder mass="2.0" length="0.125" radius="0.08">
+            <origin xyz="0 0 0.0625" rpy="0 0 0"/>
+        </xacro:inertial_cylinder>
+    </link>
+    <!-- LEFT WHEEL LINK -->
+    <joint name="left_wheel_joint" type="continuous">
+        <parent link="base_link"/>
+        <child link="left_wheel"/>
+        <origin xyz="0 0.08 0" rpy="-${pi/2} 0 0"/>
+        <axis xyz="0 0 1"/>
+    </joint>
+    <link name="left_wheel">
+        <visual>
+            <geometry>
+                <cylinder radius="0.0325" length="0.02"/>
+                <material name="black"/>
+            </geometry>
+        </visual>
+        <collision>
+            <geometry>
+                <cylinder radius="0.0325" length="0.02"/>
+            </geometry>
+        </collision>
+        <xacro:inertial_cylinder mass="0.5" length="0.02" radius="0.0325">
+            <origin xyz="0 0 0" rpy="0 0 0"/>
+        </xacro:inertial_cylinder>
+    </link>
+    <!-- RIGHT WHEEL LINK -->
+    <joint name="right_wheel_joint" type="continuous">
+        <parent link="base_link"/>
+        <child link="right_wheel"/>
+        <origin xyz="0 -0.08 0" rpy="${pi/2} 0 0"/>
+        <axis xyz="0 0 -1"/>
+    </joint>
+    <link name="right_wheel">
+        <visual>
+            <geometry>
+                <cylinder radius="0.0325" length="0.02"/>
+                <material name="black"/>
+            </geometry>
+        </visual>
+        <collision>
+            <geometry>
+                <cylinder radius="0.0325" length="0.02"/>
+            </geometry>
+        </collision>
+        <xacro:inertial_cylinder mass="0.5" length="0.02" radius="0.0325">
+            <origin xyz="0 0 0" rpy="0 0 0"/>
+        </xacro:inertial_cylinder>
+    </link>
+    <!-- Front Caster Wheel Link -->
+    <joint name="front_caster_wheel_joint" type="fixed">
+        <parent link="chassis"/>
+        <child link="front_caster_wheel"/>
+        <origin xyz="0.07 0 0"/>
+    </joint>
+    <link name="front_caster_wheel">
+        <visual>
+            <geometry>
+                <sphere radius="0.0325"/>
+            </geometry>
+            <material name="black"/>
+        </visual>
+        <collision>
+            <geometry>
+                <sphere radius="0.0325"/>
+            </geometry>
+        </collision>
+        <xacro:inertial_sphere mass="0.5" radius="0.0325">
+            <origin xyz="0 0 0" rpy="0 0 0"/>
+        </xacro:inertial_sphere>
+    </link>
+    <!-- Back Caster Wheel Link -->
+    <joint name="back_caster_wheel_joint" type="fixed">
+        <parent link="chassis"/>
+        <child link="back_caster_wheel"/>
+        <origin xyz="-0.07 0 0"/>
+    </joint>
+    <link name="back_caster_wheel">
+        <visual>
+            <geometry>
+                <sphere radius="0.0325"/>
+            </geometry>
+            <material name="black"/>
+        </visual>
+        <collision>
+            <geometry>
+                <sphere radius="0.0325"/>
+            </geometry>
+        </collision>
+        <xacro:inertial_sphere mass="0.5" radius="0.0325">
+            <origin xyz="0 0 0" rpy="0 0 0"/>
+        </xacro:inertial_sphere>
+    </link>
 </robot>
