Commit message: new gazebo update 1

File: jazzy_ws/src/blue_bot/description/gazebo_control.xacro (robot description, xacro)
@@ -6,6 +6,6 @@
             <left_joint>left_wheel_joint</left_joint>
             <right_joint>right_wheel_joint</right_joint>
-            <wheel_separation>0.35</wheel_separation>
-            <wheel_diameter>0.1</wheel_diameter>
+            <wheel_separation>0.16</wheel_separation>
+            <wheel_radius>0.08</wheel_radius>
             <!-- Limits -->
             <max_wheel_torque>200</max_wheel_torque>

File: jazzy_ws/src/blue_bot/description/robot.urdf.xacro (robot description, xacro)
@@ -2,5 +2,5 @@
 <robot xmlns:xacro="http://www.ros.org/wiki/xacro"  name="robot">
     <xacro:include filename="robot_core.xacro" />
-    <!-- <xacro:include filename="gazebo_control.xacro" /> -->
+    <xacro:include filename="gazebo_control.xacro" />
     <!-- <xacro:include filename="lidar.xacro" /> -->
     <!-- <xacro:include filename="camera.xacro" /> -->

File: jazzy_ws/src/blue_bot/description/robot_core.xacro (robot description, xacro)
@@ -115,4 +115,9 @@
         </xacro:inertial_sphere>
     </link>
+    <gazebo reference="front_caster_wheel">
+        <material>Gazebo/Black</material>
+        <mu1 value="0.001"/>
+        <mu2 value="0.001"/>
+    </gazebo>
     <!-- Back Caster Wheel Link -->
     <joint name="back_caster_wheel_joint" type="fixed">
@@ -137,3 +142,8 @@
         </xacro:inertial_sphere>
     </link>
+    <gazebo reference="back_caster_wheel">
+        <material>Gazebo/Black</material>
+        <mu1 value="0.001"/>
+        <mu2 value="0.001"/>
+    </gazebo>
 </robot>
